Commit message: fix(WF_TRON1A/B): add hub motor housing to knee collision
The wheel hub motor housing is part of the knee link mesh (radius 52 mm
around the wheel axle, y -13..43 mm in the knee frame), but no collision
geometry covered it: the knee had a thin shank rod (URDF/MJCF) or a sphere
at the knee joint (xacro), and the wheel collision only covers the tire.
Inward leg swings could therefore interpenetrate in simulation (#2).

Add a cylinder collision for the housing to knee_L/R_Link in robot.urdf,
robot.xml and the xacro sources of WF_TRON1A and WF_TRON1B.

Checked in MuJoCo 3.16 over 6,435 one-leg-adducted poses: of 391 poses
where the real housings overlap, the original model missed 201; the fixed
model catches all of them, and its extra contacts are all within 3 mm of
the real geometry. Standing pose and a 2 s drop behave the same.

Fixes #2

File: pointfoot/WF_TRON1A/urdf/robot.urdf (robot description, URDF)
Before this commit: robot wheel_biped, 10 links, 9 joints
Links:
- link knee_L_Link: geometry collision cylinder length=0.0562 radius=0.052; collision cylinder length=0.26 radius=0.015
- link knee_R_Link: geometry collision cylinder length=0.0562 radius=0.052; collision cylinder length=0.26 radius=0.015

File: pointfoot/WF_TRON1A/xacro/const.xacro (robot description, xacro)
@@ -33,4 +33,8 @@
     <xacro:property name="wheel_offset_y" value="0.0435"/>
     <xacro:property name="wheel_offset_z" value="-0.25981"/>
+    <!-- hub motor housing on the knee link, around the wheel axle (knee frame) -->
+    <xacro:property name="knee_motor_radius" value="0.052"/>
+    <xacro:property name="knee_motor_length" value="0.0562"/>
+    <xacro:property name="knee_motor_offset_y" value="0.0149"/>
     <!-- joint limits -->
     <!-- <xacro:property name="damping" value="0"/> -->

File: pointfoot/WF_TRON1A/xacro/leg.xacro (robot description, xacro)
@@ -96,4 +96,11 @@
                 </geometry>
             </collision>
+            <!-- hub motor housing around the wheel axle -->
+            <collision>
+                <origin rpy="1.570796327 0 0" xyz="${wheel_offset_x} ${knee_motor_offset_y*mirror} ${wheel_offset_z}"/>
+                <geometry>
+                    <cylinder length="${knee_motor_length}" radius="${knee_motor_radius}"/>
+                </geometry>
+            </collision>
             <inertial>
                 <origin rpy="0 0 0" xyz="${knee_com_x} ${knee_com_y*mirror} ${knee_com_z}"/>

File: pointfoot/WF_TRON1B/urdf/robot.urdf (robot description, URDF)
Before this commit: robot wheel_biped, 10 links, 9 joints
Links:
- link knee_L_Link: geometry collision cylinder length=0.0562 radius=0.052; collision cylinder length=0.26 radius=0.015
- link knee_R_Link: geometry collision cylinder length=0.0562 radius=0.052; collision cylinder length=0.26 radius=0.015

File: pointfoot/WF_TRON1B/xacro/leg.xacro (robot description, xacro)
@@ -96,4 +96,11 @@
                 </geometry>
             </collision>
+            <!-- hub motor housing around the wheel axle -->
+            <collision>
+                <origin rpy="1.570796327 0 0" xyz="${wheel_offset_x} ${knee_motor_offset_y*mirror} ${wheel_offset_z}"/>
+                <geometry>
+                    <cylinder length="${knee_motor_length}" radius="${knee_motor_radius}"/>
+                </geometry>
+            </collision>
             <inertial>
                 <origin rpy="0 0 0" xyz="${knee_com_x} ${knee_com_y*mirror} ${knee_com_z}"/>
